Commit message: exp1.5：URDF 切回 physically_mirrored + armature 按 M_ii 重校 + 删除 play_gm.py
- asset.file: X1_12DOF.urdf → X1_12DOF_physically_mirrored.urdf
- 工作区 PM.urdf 右踝 pitch 轴已改为 (0 0 1)，与 X1_12DOF 一致，config 符号沿用
- armature 恢复 exp0.1（同 URDF）验证值：髋Pitch [0.09,0.23]/髋Yaw [0.003,0.018]/膝 [0.18,0.32]
  （站姿 M_ii 变化：0.225→0.271 / 0.0265→0.0309 / 0.0883→0.1127，与辨识文档 §12 perfect_mirrored 列吻合）
- 踝 armature 覆盖随机化 [0.003,0.04] 保留；action_smoothness -0.008 沿用 exp1.4
- play.py 回放固定基准同步新范围中值（髋Yaw 0.0105/膝 0.25）
- 删除 play_gm.py（云端回放脚本弃用），replay.md 引用同步更新

File: resources/robots/x1/urdf/X1_12DOF_physically_mirrored.urdf (robot description, URDF)
Before this commit: robot X1_12DOF, 60 links, 59 joints
Joints:
- joint right_ankle_pitch_joint: axis 0 0 -1 -> 0 0 1
